File: Lab4/sch/sch.kicad_sch (KiCad schematic)
At the start: 3 parts, among them SW1 SW_Push, U1 2478, U2 Pico

Commit message: Final Version
Connections:
- net at U1.10 (Y1+): no longer U2.32 (GPIO27_ADC1)
- net at U1.11 (X1-): no longer U2.31 (GPIO26_ADC0)
- net at U1.12 (Y1-): no longer U2.27 (GPIO21)
- net at U1.27 (CS2): now also U2.24 (GPIO18)
- net at U1.29 (RST2): now also U2.26 (GPIO20)
- net at U1.31 (Y2+): now also U2.32 (GPIO27_ADC1)
- net at U1.32 (X2+): now also U2.29 (GPIO22)
- net at U1.33 (Y2-): now also U2.27 (GPIO21)
- net at U1.34 (X2-): now also U2.31 (GPIO26_ADC0)
- net at U1.39 (CCS): no longer U2.24 (GPIO18)
- net at U1.7 (RST1): no longer U2.26 (GPIO20)
- net at U1.9 (X1+): no longer U2.29 (GPIO22)
